Commit message: Update robot.xacro

File: model/robot.xacro (robot description, xacro)
@@ -1 +1,254 @@
-kk
+<?xml version="1.0"?>
+<robot name="differential_drive_robot" xmlns:xacro="http://www.ros.org/wiki/xacro">
+  <!-- ============================= -->
+  <!-- MATERIALS -->
+  <!-- ============================= -->
+   <material name="gray">
+     <!-- Base & lidar  -->
+    <color rgba='.7 .7 .7 1.0' />
+   </material>
+   <material name="black">
+    <!-- Lifter -->
+    <color rgba='0 0 0 1' />
+   </material>
+   <material name='blue'>
+    <!-- wheels -->
+    <color rgba='0 0 1 1'/>
+   </material>
+  <!-- ============================= -->
+  <!-- VARIABLES -->
+  <!-- ============================= -->
+  <xacro:property name="base_length" value="0.7"/>
+  <xacro:property name="base_width"  value="0.5"/>
+  <xacro:property name="base_height" value="0.134"/>
+  <xacro:property name="wheel_radius" value="0.0625"/>
+  <xacro:property name="wheel_width"  value="0.04"/>
+  <xacro:property name="lidar_length" value=".055"/>
+  <xacro:property name="lidar_radius" value="0.0484"/>
+  <xacro:property name="lifter_length" value=".322"/>
+  <xacro:property name="lifter_width" value=".375"/>
+  <xacro:property name="lifter_height" value=".035"/>
+<!-- ============================= -->
+  <!-- Inertia Functions -->
+  <!-- ============================= -->
+<xacro:macro name="box_inertia" params="m x y z o_xyz o_rpy">
+  <inertial>
+    <mass value="${m}" />
+    <origin xyz="${o_xyz}" rpy="${o_rpy}" />
+    <inertia
+      ixx="${(m/12) * (z*z + y*y)}"
+      ixy="0"
+      ixz="0"
+      iyy="${(m/12) * (x*x + z*z)}"
+      iyz="0"
+      izz="${(m/12) * (x*x + y*y)}"
+    />
+  </inertial>
+</xacro:macro>
+<xacro:macro name="cylinder_inertia" params="m r l o_xyz o_rpy">
+  <inertial>
+    <mass value="${m}" />
+    <origin xyz="${o_xyz}" rpy="${o_rpy}" />
+    <inertia
+      ixx="${(m/12) * (3*r*r + l*l)}"
+      ixy="0"
+      ixz="0"
+      iyy="${(m/12) * (3*r*r + l*l)}"
+      iyz="0"
+      izz="${(m/2) * (r*r)}"
+    />
+  </inertial>
+</xacro:macro>
+<!-- ============================= -->
+<!-- BASE LINK -->
+<!-- ============================= -->
+<link name="base_link">
+  <xacro:box_inertia m='4' x="${base_length}" y='${base_width}' z='${base_height}' o_xyz='0 0 ${(base_height/2)+(wheel_radius*2)}' o_rpy='0 0 0'/>
+  <visual>
+    <geometry>
+      <box size="${base_length} ${base_width} ${base_height}"/>
+    </geometry>
+    <origin xyz='0 0 ${(base_height/2)+(wheel_radius*2)}' rpy='0 0 0 '/>
+    <material name='gray'/>
+  </visual>
+  <collision>
+    <geometry>
+      <box size="${base_length} ${base_width} ${base_height}"/>
+    </geometry>
+    <origin xyz='0 0 ${(base_height/2)+(wheel_radius*2)}' rpy='0 0 0 '/>
+    <material name='gray'/>
+  </collision>
+</link>
+<!-- ============================= -->
+<!-- FOOTPRINT LINK -->
+<!-- ============================= -->
+  <link name='base_footprint'/>
+  <joint name="base_footprint_joint" type="fixed">
+  <parent link="base_footprint"/>
+  <child link="base_link"/>
+  <origin xyz="0 0 0.05" rpy="0 0 0"/>
+</joint>
+<!-- ============================= -->
+  <!-- IMU LINK -->
+  <!-- ============================= -->
+  <!-- 4 WHEELS -->
+  <!-- Back LEFT WHEEL -->
+<link name="wheel_back_left">
+    <xacro:cylinder_inertia m="0.15" r="${wheel_radius}" l="${wheel_width}" o_xyz="0 0 0" o_rpy="1.5708 0 0"/>
+    <visual>
+      <geometry>
+        <cylinder radius="${wheel_radius}" length="${wheel_width}"/>
+      </geometry>
+      <origin xyz='0 0 0' rpy='1.5708 0 0'/>
+      <material name='blue'/>
+    </visual>
+    <collision>
+      <geometry>
+        <cylinder radius="${wheel_radius}" length="${wheel_width}"/>
+      </geometry>
+      <origin xyz='0 0 0' rpy='1.5708 0 0'/>
+      <material name='blue'/>
+    </collision>
+  </link>
+  <joint name="joint_wheel_back_left" type="continuous">
+    <parent link="base_link"/>
+    <child link="wheel_back_left"/>
+    <origin xyz='-.198 ${(base_width/2)-(wheel_width/2)} ${wheel_radius}' rpy='0 0 0 '/>
+    <axis xyz="0 1 0"/>
+    <limit effort='50000' velocity='10'/>
+    <dynamics damping='1' friction='1'/>
+  </joint>
+  <!-- ============================= -->
+  <!-- Front LEFT WHEEL -->
+  <link name="wheel_front_left">
+    <xacro:cylinder_inertia m="0.15" r="${wheel_radius}" l="${wheel_width}" o_xyz="0 0 0" o_rpy="1.5708 0 0"/>
+    <visual>
+      <geometry>
+        <cylinder radius="${wheel_radius}" length="${wheel_width}"/>
+      </geometry>
+      <origin xyz='0 0 0' rpy='1.5708 0 0 '/>
+      <material name='blue'/>
+    </visual>
+    <collision>
+      <geometry>
+        <cylinder radius="${wheel_radius}" length="${wheel_width}"/>
+      </geometry>
+      <origin xyz='0 0 0' rpy='1.5708 0 0 '/>
+      <material name='blue'/>
+    </collision>
+  </link>
+  <joint name="joint_wheel_front_left" type="continuous">
+    <parent link="base_link"/>
+    <child link="wheel_front_left"/>
+    <origin xyz='.198 ${(base_width/2)-(wheel_width/2)} ${wheel_radius}' rpy='0 0 0 '/>
+    <axis xyz="0 1 0"/>
+    <limit effort='50000' velocity='10'/>
+    <dynamics damping='1' friction='1'/>
+  </joint>
+  <!-- BACK RIGHT WHEEL -->
+  <link name="wheel_back_right">
+    <xacro:cylinder_inertia m="0.15" r="${wheel_radius}" l="${wheel_width}" o_xyz="0 0 0" o_rpy="1.5708 0 0"/>
+    <visual>
+      <geometry>
+        <cylinder radius="${wheel_radius}" length="${wheel_width}"/>
+      </geometry>
+      <origin xyz='0 0 0' rpy='1.5708 0 0'/>
+      <material name='blue'/>
+    </visual>
+    <collision>
+     <geometry>
+        <cylinder radius="${wheel_radius}" length="${wheel_width}"/>
+      </geometry>
+      <origin xyz='0 0 0' rpy='1.5708 0 0'/>
+      <material name='blue'/>
+    </collision>
+  </link>
+  <joint name="joint_wheel_back_right" type="continuous">
+    <parent link="base_link"/>
+    <child link="wheel_back_right"/>
+    <origin xyz="-.198 ${-(base_width/2)+(wheel_width/2)} ${wheel_radius}" rpy="0 0 0"/>
+    <axis xyz="0 1 0"/>
+    <limit effort='50000' velocity='10'/>
+    <dynamics damping='1' friction='1'/>
+  </joint>
+<!-- Front RIGHT WHEEL -->
+  <link name="wheel_front_right">
+    <xacro:cylinder_inertia m="0.15" r="${wheel_radius}" l="${wheel_width}" o_xyz="0 0 0" o_rpy="1.5708 0 0"/>
+    <visual>
+      <geometry>
+        <cylinder radius="${wheel_radius}" length="${wheel_width}"/>
+      </geometry>
+      <origin xyz='0 0 0' rpy='1.5708 0 0'/>
+      <material name='blue'/>
+    </visual>
+    <collision>
+      <geometry>
+        <cylinder radius="${wheel_radius}" length="${wheel_width}"/>
+      </geometry>
+      <origin xyz='0 0 0' rpy='1.5708 0 0'/>
+      <material name='blue'/>
+    </collision>
+  </link>
+  <joint name="joint_wheel_front_right" type="continuous">
+    <parent link="base_link"/>
+    <child link="wheel_front_right"/>
+    <origin xyz=".198 ${-(base_width/2)+(wheel_width/2)} ${wheel_radius}" rpy="0 0 0"/>
+    <axis xyz="0 1 0"/>
+    <limit effort='50000' velocity='10'/>
+    <dynamics damping='1' friction='1'/>
+  </joint>
+  <!-- ============================= -->
+  <!-- LiDAR -->
+  <!-- ============================= -->
+  <!-- LiDAR Link -->
+<link name="laser_frame">
+  <xacro:cylinder_inertia m=".1" r="${lidar_radius}" l="${lidar_length}" o_xyz="0 0 0" o_rpy="0 0 0"/>
+  <visual>
+    <geometry>
+      <cylinder radius="${lidar_radius}" length="${lidar_length}"/>
+    </geometry>
+    <material name="black"/>
+    <origin xyz="0 0 0" rpy="0 0 0"/>
+  </visual>
+  <collision>
+    <geometry>
+      <cylinder radius="${lidar_radius}" length="${lidar_length}"/>
+    </geometry>
+    <material name="black"/>
+    <origin xyz="0 0 0" rpy="0 0 0"/>
+  </collision>
+</link>
+<joint name="laser_frame_joint" type="fixed">
+  <parent link="base_link"/>
+  <child link="laser_frame"/>
+  <origin xyz="${(base_length/2)-lidar_radius} 0 ${(base_height+(wheel_radius*2))}" rpy="0 0 0"/>
+</joint>
+  <!-- ============================= -->
+  <!-- Lifter -->
+  <!-- ============================= -->
+  <link name="lifter">
+    <visual>
+      <geometry>
+        <box size="${lifter_length} ${lifter_width} ${lifter_height}"/>
+      </geometry>
+      <material name="black"/>
+    </visual>
+    <collision>
+      <geometry>
+        <box size="${lifter_length} ${lifter_width} ${lifter_height}"/>
+      </geometry>
+    </collision>
+    <inertial>
+      <mass value="1.0"/>
+      <inertia ixx="0.01" iyy="0.01" izz="0.01" ixy="0" ixz="0" iyz="0"/>
+    </inertial>
+  </link>
+  <joint name="Lifter_Movement" type="prismatic">
+    <parent link="base_link"/>
+    <child link="lifter"/>
+    <origin xyz="0 0 ${(base_height+(wheel_radius*2))}" rpy="0 0 0"/>
+    <axis xyz="0 0 1"/>
+    <limit lower="0.0" upper="1" effort="500.0" velocity="1.0"/>
+  </joint>
+ <xacro:include filename="$(find mobile_robot)/model/robot.gazebo"/>
+</robot>
